Commit message: description

File: maze_description/urdf/drive_wheel_transmission.xacro (robot description, xacro)
@@ -9,5 +9,5 @@
       <kp value="10000000.0" />
       <kd value="1.0" />
-      <material>Gazebo/Grey</material>
+      <material>Gazebo/Black</material>
   </gazebo>
   <!-- This block connects the wheel joint to an actuator (motor), which informs both

File: maze_description/urdf/gazebo_plugin.xacro (robot description, xacro)
@@ -38,5 +38,5 @@
 <xacro:set_castor_joint_friction link="front_left_holder_link" friction="2"/>
 <xacro:set_castor_joint_friction link="back_left_holder_link" friction="2"/>
-  <!-- <gazebo reference="imu_link">
+  <gazebo reference="imu_link">
     <material>Gazebo/Grey</material>
     <sensor type="imu" name="imu">
@@ -45,5 +45,5 @@
       <visualize>true</visualize>
     </sensor>
-  </gazebo> -->
+  </gazebo>
 <!-- front lidar link -->
   <!-- <gazebo reference="back_lidar_link">

File: maze_description/urdf/main.xacro (robot description, xacro)
@@ -2,9 +2,8 @@
 <robot xmlns:xacro="http://www.ros.org/wiki/xacro" name="maze">
   <!-- xacro include     -->
-  <xacro:include filename="$(find maze_gazebo)/urdf/drive_wheel_transmission.xacro" />
-  <xacro:include filename="$(find maze_gazebo)/urdf/castor_transmission.xacro" />
-  <xacro:include filename="$(find maze_gazebo)/urdf/castor_holder_transmission.xacro" />
-  <xacro:include filename="$(find maze_gazebo)/urdf/gazebo_plugin.xacro" />
-<!--
+  <xacro:include filename="$(find maze_description)/urdf/drive_wheel_transmission.xacro" />
+  <xacro:include filename="$(find maze_description)/urdf/castor_transmission.xacro" />
+  <xacro:include filename="$(find maze_description)/urdf/castor_holder_transmission.xacro" />
+  <xacro:include filename="$(find maze_description)/urdf/gazebo_plugin.xacro" />
   <link name="base_footprint"/>
   <joint
@@ -20,10 +19,11 @@
     <axis
       xyz="0 0 0" />
-  </joint> -->
+  </joint>
+<!-- -0.0028869526654115 0.254001519517849 0.00673364367028377 -->
   <link
     name="base_link">
     <inertial>
       <origin
-        xyz="-0.0028869526654115 0.254001519517849 0.00673364367028377"
+        xyz="0 0 0.2"
         rpy="0 0 0" />
       <mass
@@ -43,19 +43,19 @@
       <geometry>
         <mesh
-          filename="package://maze_gazebo/meshes/base_link.STL" />
-      </geometry>
-      <material
-        name="">
-        <color
-          rgba="0.792156862745098 0.819607843137255 0.933333333333333 1" />
-      </material>
-    </visual>
-    <collision>
-      <origin
-        xyz="0 0 0"
-        rpy="0 0 0" />
-      <geometry>
-        <mesh
-          filename="package://maze_gazebo/meshes/base_link.STL" />
+          filename="package://maze_description/meshes/base_link.STL" />
+      </geometry>
+      <material
+        name="">
+        <color
+          rgba="0.792156862745098 0.819607843137255 0.933333333333333 1" />
+      </material>
+    </visual>
+    <collision>
+      <origin
+        xyz="0 0 0"
+        rpy="0 0 0" />
+      <geometry>
+        <mesh
+          filename="package://maze_description/meshes/base_link.STL" />
       </geometry>
     </collision>
@@ -97,19 +97,19 @@
       <geometry>
         <mesh
-          filename="package://maze_gazebo/meshes/left_wheel_link.STL" />
-      </geometry>
-      <material
-        name="">
-        <color
-          rgba="0.792156862745098 0.819607843137255 0.933333333333333 1" />
-      </material>
-    </visual>
-    <collision>
-      <origin
-        xyz="0 0 0"
-        rpy="0 0 0" />
-      <geometry>
-        <mesh
-          filename="package://maze_gazebo/meshes/left_wheel_link.STL" />
+          filename="package://maze_description/meshes/left_wheel_link.STL" />
+      </geometry>
+      <material
+        name="">
+        <color
+          rgba="0.792156862745098 0.819607843137255 0.933333333333333 1" />
+      </material>
+    </visual>
+    <collision>
+      <origin
+        xyz="0 0 0"
+        rpy="0 0 0" />
+      <geometry>
+        <mesh
+          filename="package://maze_description/meshes/left_wheel_link.STL" />
       </geometry>
     </collision>
@@ -150,19 +150,19 @@
       <geometry>
         <mesh
-          filename="package://maze_gazebo/meshes/right_wheel_link.STL" />
-      </geometry>
-      <material
-        name="">
-        <color
-          rgba="0.792156862745098 0.819607843137255 0.933333333333333 1" />
-      </material>
-    </visual>
-    <collision>
-      <origin
-        xyz="0 0 0"
-        rpy="0 0 0" />
-      <geometry>
-        <mesh
-          filename="package://maze_gazebo/meshes/right_wheel_link.STL" />
+          filename="package://maze_description/meshes/right_wheel_link.STL" />
+      </geometry>
+      <material
+        name="">
+        <color
+          rgba="0.792156862745098 0.819607843137255 0.933333333333333 1" />
+      </material>
+    </visual>
+    <collision>
+      <origin
+        xyz="0 0 0"
+        rpy="0 0 0" />
+      <geometry>
+        <mesh
+          filename="package://maze_description/meshes/right_wheel_link.STL" />
       </geometry>
     </collision>
@@ -203,19 +203,19 @@
       <geometry>
         <mesh
-          filename="package://maze_gazebo/meshes/front_left_holder_link.STL" />
-      </geometry>
-      <material
-        name="">
-        <color
-          rgba="0.792156862745098 0.819607843137255 0.933333333333333 1" />
-      </material>
-    </visual>
-    <collision>
-      <origin
-        xyz="0 0 0"
-        rpy="0 0 0" />
-      <geometry>
-        <mesh
-          filename="package://maze_gazebo/meshes/front_left_holder_link.STL" />
+          filename="package://maze_description/meshes/front_left_holder_link.STL" />
+      </geometry>
+      <material
+        name="">
+        <color
+          rgba="0.792156862745098 0.819607843137255 0.933333333333333 1" />
+      </material>
+    </visual>
+    <collision>
+      <origin
+        xyz="0 0 0"
+        rpy="0 0 0" />
+      <geometry>
+        <mesh
+          filename="package://maze_description/meshes/front_left_holder_link.STL" />
       </geometry>
     </collision>
@@ -232,5 +232,5 @@
       link="front_left_holder_link" />
     <axis
-      xyz="0 0 1" />
+      xyz="0 1 0" />
   </joint>
   <link
@@ -256,19 +256,19 @@
       <geometry>
         <mesh
-          filename="package://maze_gazebo/meshes/front_left_castor_link.STL" />
-      </geometry>
-      <material
-        name="">
-        <color
-          rgba="0.792156862745098 0.819607843137255 0.933333333333333 1" />
-      </material>
-    </visual>
-    <collision>
-      <origin
-        xyz="0 0 0"
-        rpy="0 0 0" />
-      <geometry>
-        <mesh
-          filename="package://maze_gazebo/meshes/front_left_castor_link.STL" />
+          filename="package://maze_description/meshes/front_left_castor_link.STL" />
+      </geometry>
+      <material
+        name="">
+        <color
+          rgba="0.792156862745098 0.819607843137255 0.933333333333333 1" />
+      </material>
+    </visual>
+    <collision>
+      <origin
+        xyz="0 0 0"
+        rpy="0 0 0" />
+      <geometry>
+        <mesh
+          filename="package://maze_description/meshes/front_left_castor_link.STL" />
       </geometry>
     </collision>
@@ -285,5 +285,5 @@
       link="front_left_castor_link" />
     <axis
-      xyz="0 1 0" />
+      xyz="0 0 1" />
   </joint>
   <link
@@ -309,19 +309,19 @@
       <geometry>
         <mesh
-          filename="package://maze_gazebo/meshes/front_right_holder_link.STL" />
-      </geometry>
-      <material
-        name="">
-        <color
-          rgba="0.792156862745098 0.819607843137255 0.933333333333333 1" />
-      </material>
-    </visual>
-    <collision>
-      <origin
-        xyz="0 0 0"
-        rpy="0 0 0" />
-      <geometry>
-        <mesh
-          filename="package://maze_gazebo/meshes/front_right_holder_link.STL" />
+          filename="package://maze_description/meshes/front_right_holder_link.STL" />
+      </geometry>
+      <material
+        name="">
+        <color
+          rgba="0.792156862745098 0.819607843137255 0.933333333333333 1" />
+      </material>
+    </visual>
+    <collision>
+      <origin
+        xyz="0 0 0"
+        rpy="0 0 0" />
+      <geometry>
+        <mesh
+          filename="package://maze_description/meshes/front_right_holder_link.STL" />
       </geometry>
     </collision>
@@ -338,5 +338,5 @@
       link="front_right_holder_link" />
     <axis
-      xyz="0 0 1" />
+      xyz="0 1 0" />
   </joint>
   <link
@@ -362,19 +362,19 @@
       <geometry>
         <mesh
-          filename="package://maze_gazebo/meshes/front_right_castor_link.STL" />
-      </geometry>
-      <material
-        name="">
-        <color
-          rgba="0.792156862745098 0.819607843137255 0.933333333333333 1" />
-      </material>
-    </visual>
-    <collision>
-      <origin
-        xyz="0 0 0"
-        rpy="0 0 0" />
-      <geometry>
-        <mesh
-          filename="package://maze_gazebo/meshes/front_right_castor_link.STL" />
+          filename="package://maze_description/meshes/front_right_castor_link.STL" />
+      </geometry>
+      <material
+        name="">
+        <color
+          rgba="0.792156862745098 0.819607843137255 0.933333333333333 1" />
+      </material>
+    </visual>
+    <collision>
+      <origin
+        xyz="0 0 0"
+        rpy="0 0 0" />
+      <geometry>
+        <mesh
+          filename="package://maze_description/meshes/front_right_castor_link.STL" />
       </geometry>
     </collision>
@@ -391,5 +391,5 @@
       link="front_right_castor_link" />
     <axis
-      xyz="0 1 0" />
+      xyz="0 0 1" />
   </joint>
   <link
@@ -415,19 +415,19 @@
       <geometry>
         <mesh
-          filename="package://maze_gazebo/meshes/back_left_holder_link.STL" />
-      </geometry>
-      <material
-        name="">
-        <color
-          rgba="0.792156862745098 0.819607843137255 0.933333333333333 1" />
-      </material>
-    </visual>
-    <collision>
-      <origin
-        xyz="0 0 0"
-        rpy="0 0 0" />
-      <geometry>
-        <mesh
-          filename="package://maze_gazebo/meshes/back_left_holder_link.STL" />
+          filename="package://maze_description/meshes/back_left_holder_link.STL" />
+      </geometry>
+      <material
+        name="">
+        <color
+          rgba="0.792156862745098 0.819607843137255 0.933333333333333 1" />
+      </material>
+    </visual>
+    <collision>
+      <origin
+        xyz="0 0 0"
+        rpy="0 0 0" />
+      <geometry>
+        <mesh
+          filename="package://maze_description/meshes/back_left_holder_link.STL" />
       </geometry>
     </collision>
@@ -444,5 +444,5 @@
       link="back_left_holder_link" />
     <axis
-      xyz="0 0 1" />
+      xyz="0 1 0" />
   </joint>
   <link
@@ -468,19 +468,19 @@
       <geometry>
         <mesh
-          filename="package://maze_gazebo/meshes/back_left_castor_link.STL" />
-      </geometry>
-      <material
-        name="">
-        <color
-          rgba="0.792156862745098 0.819607843137255 0.933333333333333 1" />
-      </material>
-    </visual>
-    <collision>
-      <origin
-        xyz="0 0 0"
-        rpy="0 0 0" />
-      <geometry>
-        <mesh
-          filename="package://maze_gazebo/meshes/back_left_castor_link.STL" />
+          filename="package://maze_description/meshes/back_left_castor_link.STL" />
+      </geometry>
+      <material
+        name="">
+        <color
+          rgba="0.792156862745098 0.819607843137255 0.933333333333333 1" />
+      </material>
+    </visual>
+    <collision>
+      <origin
+        xyz="0 0 0"
+        rpy="0 0 0" />
+      <geometry>
+        <mesh
+          filename="package://maze_description/meshes/back_left_castor_link.STL" />
       </geometry>
     </collision>
@@ -497,5 +497,5 @@
       link="back_left_castor_link" />
     <axis
-      xyz="0 1 0" />
+      xyz="0 0 1" />
   </joint>
   <link
@@ -521,19 +521,19 @@
       <geometry>
         <mesh
-          filename="package://maze_gazebo/meshes/back_right_holder_link.STL" />
-      </geometry>
-      <material
-        name="">
-        <color
-          rgba="0.792156862745098 0.819607843137255 0.933333333333333 1" />
-      </material>
-    </visual>
-    <collision>
-      <origin
-        xyz="0 0 0"
-        rpy="0 0 0" />
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