Commit message: world

File: maze_description/urdf/gazebo_plugin.xacro (robot description, xacro)
@@ -16,5 +16,5 @@
       <minDepth>0.001</minDepth>
       <fdir1>0 0 0</fdir1>
-      <max_vel>1</max_vel>
+      <max_vel>0.5</max_vel>
     </gazebo>
   </xacro:macro>
@@ -26,16 +26,16 @@
   </xacro:macro>
 <!-- friction for drive wheels -->
-<xacro:set_wheel_friction link="left_wheel_link" friction="10"/>
-<xacro:set_wheel_friction link="right_wheel_link" friction="10"/>
+<xacro:set_wheel_friction link="left_wheel_link" friction="1"/>
+<xacro:set_wheel_friction link="right_wheel_link" friction="1"/>
 <!-- friction for caster wheels -->
-<xacro:set_wheel_friction link="front_right_castor_link" friction="0.1"/>
-<xacro:set_wheel_friction link="back_right_castor_link" friction="0.1"/>
-<xacro:set_wheel_friction link="front_left_castor_link" friction="0.1"/>
-<xacro:set_wheel_friction link="back_left_castor_link" friction="0.1"/>
+<xacro:set_wheel_friction link="front_right_castor_link" friction="100000"/>
+<xacro:set_wheel_friction link="back_right_castor_link" friction="100000"/>
+<xacro:set_wheel_friction link="front_left_castor_link" friction="100000"/>
+<xacro:set_wheel_friction link="back_left_castor_link" friction="100000"/>
 <!-- friction for caster handle -->
-<xacro:set_castor_joint_friction link="front_right_holder_link" friction="2"/>
-<xacro:set_castor_joint_friction link="back_right_holder_link" friction="2"/>
-<xacro:set_castor_joint_friction link="front_left_holder_link" friction="2"/>
-<xacro:set_castor_joint_friction link="back_left_holder_link" friction="2"/>
+<xacro:set_castor_joint_friction link="front_right_holder_link" friction="100"/>
+<xacro:set_castor_joint_friction link="back_right_holder_link" friction="100"/>
+<xacro:set_castor_joint_friction link="front_left_holder_link" friction="100"/>
+<xacro:set_castor_joint_friction link="back_left_holder_link" friction="100"/>
   <gazebo reference="imu_link">
     <material>Gazebo/Grey</material>

File: maze_description/urdf/main.xacro (robot description, xacro)
@@ -25,8 +25,8 @@
     <inertial>
       <origin
-        xyz="0 0 0.2"
-        rpy="0 0 0" />
-      <mass
-        value="100" />
+        xyz="0 0.041 0.2"
+        rpy="0 0 0" />
+      <mass
+        value="200" />
       <inertia
         ixx="0.3678033044408"
@@ -82,5 +82,5 @@
         rpy="0 0 0" />
       <mass
-        value="10" />
+        value="100" />
       <inertia
         ixx="0.000414738647732841"
@@ -126,5 +126,5 @@
       link="left_wheel_link" />
     <axis
-      xyz="0 1 0" />
+      xyz="0 -1 0" />
   </joint>
   <link
@@ -135,5 +135,5 @@
         rpy="0 0 0" />
       <mass
-        value="10" />
+        value="100" />
       <inertia
         ixx="0.000414738647732841"
@@ -188,5 +188,5 @@
         rpy="0 0 0" />
       <mass
-        value="5" />
+        value="50" />
       <inertia
         ixx="0.000188864689361723"
@@ -241,5 +241,5 @@
         rpy="0 0 0" />
       <mass
-        value="5" />
+        value="20" />
       <inertia
         ixx="0.000389246550993186"
@@ -294,5 +294,5 @@
         rpy="0 0 0" />
       <mass
-        value="5" />
+        value="50" />
       <inertia
         ixx="0.000188864689908781"
@@ -347,5 +347,5 @@
         rpy="0 0 0" />
       <mass
-        value="5" />
+        value="20" />
       <inertia
         ixx="0.000389246550993186"
@@ -400,5 +400,5 @@
         rpy="0 0 0" />
       <mass
-        value="5" />
+        value="50" />
       <inertia
         ixx="0.000188864689908782"
@@ -453,5 +453,5 @@
         rpy="0 0 0" />
       <mass
-        value="5" />
+        value="20" />
       <inertia
         ixx="0.000389246550993186"
@@ -506,5 +506,5 @@
         rpy="0 0 0" />
       <mass
-        value="5" />
+        value="50" />
       <inertia
         ixx="0.000188864380636178"
@@ -559,5 +559,5 @@
         rpy="0 0 0" />
       <mass
-        value="5" />
+        value="20" />
       <inertia
         ixx="0.000389246550993186"
